File: HardwareDesign/THC-schematic.sch (EAGLE design)
At the start: 41 parts

Commit message: Rev C Hardware
Parts:
- removed ARDUNIO-COMM: JJ, pinhead:PINHD-1X6
- removed BUTTONS: CON1, pinhead:PINHD-1X6/90
- removed MEGA-IO: ARDUINO-MEGA-18X2, ArduinoConnect18x2:ARDUINO-MEGA-18X2
- removed OK4: 6N137, optocoupler:6N137
- removed R20, R21: 560, resistor:R-US_0204/5
- removed SP: 0, resistor:C-US025-025X050
- removed TO-CNC: CON3, pinhead:PINHD-1X6/90
- removed TO-PLASMA: J1, pinhead:PINHD-1X8
- removed U$2: LT1632, ArduinoThcOpAmp:LT1632
- added ARD-ANALOG, ARD-PWM, JP1: (no value), pinhead:PINHD-1X8
- added ARD-PWR: (no value), pinhead:PINHD-1X6
- added C10: 100nF / .1 uF, resistor:C-US025-025X050
- added C11: 100 nF / .1 uF, resistor:C-US025-025X050
- added CNC, TORCH: (no value), con-subd:F09HPS
- added IC1: 7805T, adafruit:7805T
- added ILQ2: ILQ1, optocoupler:ILQ1
- added J1: 2.1MM-PLUG-PCB-MNT, ArdunioPowerJack:2.1MM-PLUG-PCB-MNT
- added JP2, RELAY: (no value), pinhead:PINHD-1X3
- added R3, R4: 1k, resistor:R-US_0207/7
- C1: value .1uF -> 100 nF / 0.1uF
- C2: value 150n -> 15pf
- C3: value 1u -> 150 nf
- C4: value 10uF -> 100 nf / 0.1 uF
- C5: value 100n -> 15pf
- C6: value 100n -> 100 nF / 0.1uF
- C7: value .1uF -> 1 uF
- C8: value 15pf -> 10 uF
- C9: value 15pf -> 100 nf
- OK2: value ILQ1 -> 6N137; device optocoupler:ILQ1 -> optocoupler:6N137
- R1: value 350 -> 220k; device resistor:R-US_0204/5 -> resistor:R-US_0207/7
- R10, R11, R12: value 1k -> 560; device resistor:R-US_0204/5 -> resistor:R-US_0207/7
- R13: value 220k -> 1k; device resistor:R-US_0204/5 -> resistor:R-US_0207/7
- R14: value 15k -> 560; device resistor:R-US_0204/5 -> resistor:R-US_0207/7
- R15: value 7.87k -> 2.61k; device resistor:R-US_0204/5 -> resistor:R-US_0207/7
- R16: value 21.5k -> 560; device resistor:R-US_0204/5 -> resistor:R-US_0207/7
- R17: value 2.61k -> 350; device resistor:R-US_0204/5 -> resistor:R-US_0207/7
- R18, R19, R6: device resistor:R-US_0204/5 -> resistor:R-US_0207/7
- R2: value 350 -> 15k; device resistor:R-US_0204/5 -> resistor:R-US_0207/7
- R5: value 560 -> 1k; device resistor:R-US_0204/5 -> resistor:R-US_0207/7
- R7: value 560 -> 7.87k; device resistor:R-US_0204/5 -> resistor:R-US_0207/7
- R8: value 560 -> 350; device resistor:R-US_0204/5 -> resistor:R-US_0207/7
- R9: value 1k -> 21.5k; device resistor:R-US_0204/5 -> resistor:R-US_0207/7
- U$1: value PIN-ARD-A8 -> LT1632; device Rege:PIN-ARD-A8 -> ArduinoThcOpAmp:LT1632
Connections:
- removed net N$14: BUTTONS.1, MEGA-IO.D-33
- removed net N$15: BUTTONS.2, MEGA-IO.D-35
- removed net N$17: MEGA-IO.D-50, OK2B.C
- removed net N$18: MEGA-IO.D-48, OK2C.C
- removed net N$19: MEGA-IO.D-46, OK2D.C
- removed net N$23: BUTTONS.3, MEGA-IO.D-37
- removed net N$24: BUTTONS.4, MEGA-IO.D-39
- removed net N$25: BUTTONS.5, MEGA-IO.D-41
- removed net N$28: C4.1, R19.1, U$1.8
- new net +3.3V: ARD-PWR.5, JP2.3
- new net ARC-GOOD-ARD: ILQ2B.C, JP1.3
- new net ARD-ANALOG-IN: ARD-ANALOG.1, C8.1, R19.1
- new net N$1: C10.1, IC1.VI, J1.P$POS
- new net TORCH-DOWN-ARD: ILQ2D.C, JP1.5
- new net TORCH-UP-ARD: ILQ2C.C, JP1.4
- new net VCC: C1.1, JP2.2, OK2.VCC, R10.2, R11.2, R12.2, R13.2, R14.1, R8.1, U$1.+5
- net +5V: now also ARD-PWR.4, C11.1, IC1.VO, JP2.1, RELAY.1; no longer C1.1, MEGA-IO.+5, MEGA-IO.+5V, OK4.VCC, R12.2, R2.1, R20.1, R5.2, R6.2, R7.2, TO-PLASMA.8, U$2.+5
- net ARC-OK-INT: now also ARD-PWM.4, TORCH-7.F; no longer ARDUNIO-COMM.2, TO-PLASMA.4
- net ARDUINO-RX: now also C2.1, JP1.1, OK2.VO, R8.2; no longer ARDUNIO-COMM.3, C9.1, OK4.VO, R2.2
- net ARDUINO-TX: now also JP1.2; no longer ARDUNIO-COMM.4
- net CNC-GND: now also CNC-2.F, ILQ2B.EMIT, ILQ2C.EMIT, ILQ2D.EMIT; no longer OK2B.EMIT, OK2C.EMIT, OK2D.EMIT, TO-CNC.6
- net DIVIDER: now also R1.2, R2.2, R7.1; no longer R13.2, R14.2, R15.1, SP.1
- net GND: now also ARD-PWM.2, ARD-PWR.2, ARD-PWR.3, C10.2, C11.2, C2.2, C8.2, CNC-G.G1, IC1.GND, ILQ2A.EMIT, J1.P$NEG, J1.P$SHLD, OK2.GND, R2.1, RELAY.2, TORCH-5.F, TORCH-6.F, TORCH-G.G1, U$1.GND; no longer BUTTONS.6, C5.2, C6.2, MEGA-IO.GND, MEGA-IO.GND-, OK2A.EMIT, OK4.GND, R14.1, SP.2, TO-PLASMA.1, TO-PLASMA.5, TO-PLASMA.7, U$2.GND
- net N$10: now also CNC-5.F, ILQ2B.COL, R5.2; no longer OK2B.COL, R9.2, TO-CNC.3
- net N$11: now also CNC-4.F, ILQ2C.COL, R4.2; no longer OK2C.COL, R10.2, TO-CNC.4
- net N$12: now also CNC-3.F, ILQ2D.COL, R3.2; no longer OK2D.COL, R11.2, TO-CNC.5
- net N$16: now also CNC-6.F, ILQ2A.C; no longer OK2A.C, TO-CNC.2
- net N$2: now also ILQ2B.A, R12.1; no longer OK2B.A, R5.1
- net N$22: now also CNC-7.F, R3.1, R4.1, R5.1, R6.1; no longer R10.1, R11.1, R8.1, R9.1, TO-CNC.1
- net N$26: now also C3.2, R7.2, R9.1; no longer C2.2, R15.2, R16.1
- net N$27: now also C4.1, R9.2, U$1.+A; no longer C5.1, R16.2, U$2.+A
- net N$29: now also C3.1, R15.1, U$1.-A, U$1.OUTA; no longer C2.1, R17.1, U$2.-A, U$2.OUTA
- net N$30: now also C7.1, R15.2; no longer C3.1, R17.2
- net N$31: now also C9.1, U$1.+B; no longer C6.1, U$2.+B
- net N$32: now also R14.2; no longer R20.2
- net N$34: now also OK2.A, R16.1; no longer OK4.A, R21.1
- net N$7: now also ILQ2C.A, R11.1; no longer OK2C.A, R6.1
- net N$8: now also ILQ2D.A, R10.1; no longer OK2D.A, R7.1
- net N$9: now also ILQ2A.A, R6.2; no longer OK2A.A, R8.2
- net SERIAL+5V: now also C6.1, R16.2, R17.1; no longer C7.1, R1.1, R21.2
- net SERIAL-GND: now also C5.2, C6.2; no longer C7.2, C8.2
- net TORCH+: now also R1.1, TORCH-1.F; no longer R13.1, TO-PLASMA.2
- net TORCH-ON-INT: now also ARD-PWM.3, ILQ2A.COL, R13.1; no longer ARDUNIO-COMM.1, OK2A.COL, R12.1
- net TORCH-ON-RELAY: now also ARD-PWM.5, RELAY.3; no longer ARDUNIO-COMM.5, TO-PLASMA.6
- net UNFILTERED: now also C7.2, U$1.-B, U$1.OUTB; no longer C3.2, U$1.14, U$2.-B, U$2.OUTB
- net USB-RX: now also C5.1, R17.2; no longer C8.1, R1.2
- net USB-TX: now also OK2.C; no longer OK4.C
Other:
- note added: "ArduinoTHC Rev C"
- note added: "TORCH-"
- note added: "To CNC"
- note added: "To Plasma"
- note removed: "ArduinoTHC Rev B"
- moved on the sheet: C2, C3, C4, C5, C6, C7, C8, C9, R1, R10, R11, R12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
